Commit message: Stage 2: Search field with blue targets and random red zone
- Replace corridor with 30x40m field with yellow boundary walls
- 5 blue 1x1m ground targets at fixed positions
- Random red 8x4m no-go zone spawned each launch
- Downward-facing 2D RGB camera (removed depth cam + ToFs)
- GPS sensor retained
- Updated README, HANDOFF_ISSUES.md, entrypoint for Stage 2
- Removed test scripts (candidates write their own)

File: ros2_ws/src/drone_corridor_sim/urdf/sjtu_drone_extended.urdf.xacro (robot description, xacro)
@@ -4,6 +4,6 @@
   <!-- Base drone (has GPS via built-in plugin, IMU, sonar, flight dynamics) -->
   <xacro:include filename="$(find sjtu_drone_description)/urdf/sjtu_drone.urdf.xacro"/>
-  <!-- ── FRONT DEPTH CAMERA (simulates SC-DepthV3) ──────────── -->
-  <link name="depth_camera_link">
+  <!-- ── DOWNWARD-FACING 2D RGB CAMERA ────────────────────── -->
+  <link name="downward_cam_link">
     <inertial>
       <mass value="0.001"/>
@@ -11,109 +11,35 @@
     </inertial>
   </link>
-  <joint name="depth_camera_joint" type="fixed">
+  <joint name="downward_cam_joint" type="fixed">
     <parent link="base_link"/>
-    <child  link="depth_camera_link"/>
-    <origin xyz="0.18 0.0 0.04" rpy="0 0 0"/>
+    <child  link="downward_cam_link"/>
+    <!-- Mounted underneath, pointing straight down (pitch -90°) -->
+    <origin xyz="0.0 0.0 -0.05" rpy="0 1.5707963 0"/>
   </joint>
-  <gazebo reference="depth_camera_link">
-    <sensor name="front_depth_camera" type="depth">
+  <gazebo reference="downward_cam_link">
+    <sensor name="downward_camera" type="camera">
       <always_on>true</always_on>
       <update_rate>15</update_rate>
-      <visualize>false</visualize>
+      <visualize>true</visualize>
       <camera>
-        <horizontal_fov>1.3963</horizontal_fov>
+        <horizontal_fov>1.5708</horizontal_fov>  <!-- 90° FOV -->
         <image>
-          <width>320</width>
-          <height>240</height>
+          <width>640</width>
+          <height>480</height>
           <format>R8G8B8</format>
         </image>
         <clip>
           <near>0.1</near>
-          <far>10.0</far>
+          <far>50.0</far>
         </clip>
       </camera>
-      <plugin name="depth_camera_plugin" filename="libgazebo_ros_camera.so">
+      <plugin name="downward_cam_plugin" filename="libgazebo_ros_camera.so">
         <ros>
           <namespace>/drone</namespace>
-          <remapping>~/image_raw:=camera/image_raw</remapping>
-          <remapping>~/camera_info:=camera/camera_info</remapping>
-          <remapping>~/depth/image_raw:=camera/depth</remapping>
-          <remapping>~/depth/camera_info:=camera/depth/camera_info</remapping>
-          <remapping>~/points:=camera/points</remapping>
+          <remapping>~/image_raw:=downward_cam/image_raw</remapping>
+          <remapping>~/camera_info:=downward_cam/camera_info</remapping>
         </ros>
-        <camera_name>front_depth</camera_name>
-        <frame_name>depth_camera_link</frame_name>
-        <min_depth>0.1</min_depth>
-        <max_depth>10.0</max_depth>
-      </plugin>
-    </sensor>
-  </gazebo>
-  <!-- ── LEFT ToF (invisible) ────────────────────────────────── -->
-  <link name="tof_left_link">
-    <inertial>
-      <mass value="0.001"/>
-      <inertia ixx="1e-7" ixy="0" ixz="0" iyy="1e-7" iyz="0" izz="1e-7"/>
-    </inertial>
-  </link>
-  <joint name="tof_left_joint" type="fixed">
-    <parent link="base_link"/>
-    <child  link="tof_left_link"/>
-    <origin xyz="0.0 0.12 0.0" rpy="0 0 1.5707963"/>
-  </joint>
-  <gazebo reference="tof_left_link">
-    <sensor name="tof_left" type="ray">
-      <always_on>true</always_on>
-      <update_rate>20</update_rate>
-      <visualize>true</visualize>
-      <ray>
-        <scan>
-          <horizontal><samples>1</samples><resolution>1</resolution>
-            <min_angle>0</min_angle><max_angle>0</max_angle></horizontal>
-        </scan>
-        <range><min>0.05</min><max>3.0</max><resolution>0.01</resolution></range>
-        <noise><type>gaussian</type><mean>0</mean><stddev>0.005</stddev></noise>
-      </ray>
-      <plugin name="tof_left_plugin" filename="libgazebo_ros_ray_sensor.so">
-        <ros><namespace>/drone</namespace><remapping>~/out:=tof/left</remapping></ros>
-        <output_type>sensor_msgs/Range</output_type>
-        <radiation_type>infrared</radiation_type>
-        <frame_name>tof_left_link</frame_name>
-        <min_range>0.05</min_range><max_range>3.0</max_range>
-        <field_of_view>0.01</field_of_view>
-      </plugin>
-    </sensor>
-  </gazebo>
-  <!-- ── RIGHT ToF (invisible) ───────────────────────────────── -->
-  <link name="tof_right_link">
-    <inertial>
-      <mass value="0.001"/>
-      <inertia ixx="1e-7" ixy="0" ixz="0" iyy="1e-7" iyz="0" izz="1e-7"/>
-    </inertial>
-  </link>
-  <joint name="tof_right_joint" type="fixed">
-    <parent link="base_link"/>
-    <child  link="tof_right_link"/>
-    <origin xyz="0.0 -0.12 0.0" rpy="0 0 -1.5707963"/>
-  </joint>
-  <gazebo reference="tof_right_link">
-    <sensor name="tof_right" type="ray">
-      <always_on>true</always_on>
-      <update_rate>20</update_rate>
-      <visualize>true</visualize>
-      <ray>
-        <scan>
-          <horizontal><samples>1</samples><resolution>1</resolution>
-            <min_angle>0</min_angle><max_angle>0</max_angle></horizontal>
-        </scan>
-        <range><min>0.05</min><max>3.0</max><resolution>0.01</resolution></range>
-        <noise><type>gaussian</type><mean>0</mean><stddev>0.005</stddev></noise>
-      </ray>
-      <plugin name="tof_right_plugin" filename="libgazebo_ros_ray_sensor.so">
-        <ros><namespace>/drone</namespace><remapping>~/out:=tof/right</remapping></ros>
-        <output_type>sensor_msgs/Range</output_type>
-        <radiation_type>infrared</radiation_type>
-        <frame_name>tof_right_link</frame_name>
-        <min_range>0.05</min_range><max_range>3.0</max_range>
-        <field_of_view>0.01</field_of_view>
+        <camera_name>downward_cam</camera_name>
+        <frame_name>downward_cam_link</frame_name>
       </plugin>
     </sensor>
